File: Production Files/BigEasyDriver-GiantPanel-v16.brd (EAGLE design)
At the start: 325.6 x 168.1 mm, 2206 parts, among them IC1 A4983ALT1, IC10 A4983ALT1, IC11 LM317L, IC12 A4983ALT1, IC13 LM317L, IC14 A4983ALT1, IC15 LM317L, IC16 A4983ALT1, IC17 LM317L, IC18 A4983ALT1, IC19 LM317L, IC2 LM317L, IC20 A4983ALT1, IC21 LM317L, IC22 A4983ALT1, IC23 LM317L, IC24 A4983ALT1, IC25 LM317L, IC26 A4983ALT1, IC27 LM317L, IC28 A4983ALT1, IC29 LM317L, IC3 LM317L, IC30 A4983ALT1, IC31 LM317L, IC32 A4983ALT1, IC33 LM317L, IC34 A4983ALT1, IC35 LM317L, IC36 A4983ALT1, IC37 LM317L, IC38 A4983ALT1, IC39 LM317L, IC4 A4983ALT1, IC40 A4983ALT1, IC41 LM317L, IC42 A4983ALT1, IC43 LM317L, IC44 A4983ALT1, IC45 LM317L, IC46 A4983ALT1, IC47 LM317L, IC48 A4983ALT1, IC49 LM317L, IC5 LM317L, IC50 A4983ALT1, IC51 LM317L, IC52 A4983ALT1, IC53 LM317L, IC54 A4983ALT1, IC55 LM317L, IC56 A4983ALT1, IC57 LM317L, IC58 A4983ALT1, IC59 LM317L, IC6 A4983ALT1, IC60 A4983ALT1, IC61 LM317L, IC62 A4983ALT1, IC63 LM317L, IC64 A4983ALT1, IC65 LM317L, IC66 A4983ALT1, IC67 LM317L, IC68 A4983ALT1, IC69 LM317L, IC7 LM317L, IC70 A4983ALT1, IC71 LM317L, IC72 A4983ALT1, IC73 LM317L, IC74 A4983ALT1, IC75 LM317L, IC76 A4983ALT1, IC77 LM317L, IC78 A4983ALT1, IC79 LM317L, IC8 A4983ALT1, IC80 A4983ALT1, IC9 LM317L

Commit message: re-cammed giant panel
I made a mistake on my first cam job. Forgot that it was a 4-layer
board. This corrects that and gets the right gerbers to Gold Phoenix.
Routing:
- net V+35: track 12.3 -> 58.8 mm
- net V+31: track 12.3 -> 58.8 mm
- net V+39: track 12.3 -> 58.8 mm
- net V+32: track 12.3 -> 58.8 mm
- net V+27: track 12.3 -> 58.8 mm
- net V+23: track 12.3 -> 58.8 mm
- net V+34: track 12.3 -> 58.8 mm
- net V+33: track 12.3 -> 58.8 mm
- net V+37: track 12.3 -> 58.8 mm
- net V+28: track 12.3 -> 58.8 mm
- net V+21: track 12.3 -> 58.8 mm
- net V+38: track 12.3 -> 58.8 mm
- net V+36: track 12.3 -> 58.8 mm
- net V+30: track 12.3 -> 58.8 mm
- net V+29: track 12.3 -> 58.8 mm
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- added copper zone on layer 15, net GND20
- added copper zone on layer 15, net GND21
- added copper zone on layer 15, net GND22
- added copper zone on layer 15, net GND23
- added copper zone on layer 15, net GND24
- added copper zone on layer 15, net GND25
- added copper zone on layer 15, net GND26
- added copper zone on layer 15, net GND27
- added copper zone on layer 15, net GND28
- added copper zone on layer 15, net GND29
- added copper zone on layer 15, net GND30
- added copper zone on layer 15, net GND31
- added copper zone on layer 15, net GND32
- added copper zone on layer 15, net GND33
- added copper zone on layer 15, net GND34
- added copper zone on layer 15, net GND35
- added copper zone on layer 15, net GND36
- added copper zone on layer 15, net GND37
- added copper zone on layer 15, net GND38
- added copper zone on layer 15, net GND39
- added copper zone on layer 2, net VCC20
- added copper zone on layer 2, net VCC21
- added copper zone on layer 2, net VCC22
- added copper zone on layer 2, net VCC23
- added copper zone on layer 2, net VCC24
- added copper zone on layer 2, net VCC25
- added copper zone on layer 2, net VCC26
- added copper zone on layer 2, net VCC27
- added copper zone on layer 2, net VCC28
- added copper zone on layer 2, net VCC29
- added copper zone on layer 2, net VCC30
- added copper zone on layer 2, net VCC31
- added copper zone on layer 2, net VCC32
- added copper zone on layer 2, net VCC33
- added copper zone on layer 2, net VCC34
- added copper zone on layer 2, net VCC35
- added copper zone on layer 2, net VCC36
- added copper zone on layer 2, net VCC37
- added copper zone on layer 2, net VCC38
- added copper zone on layer 2, net VCC39
