File: Production_Files/BigEasyDriver_GiantPanel_v16a.brd (EAGLE design)
At the start: 325.6 x 168.1 mm, 2206 parts, among them IC1 A4983ALT1, IC10 A4983ALT1, IC11 LM317L, IC12 A4983ALT1, IC13 LM317L, IC14 A4983ALT1, IC15 LM317L, IC16 A4983ALT1, IC17 LM317L, IC18 A4983ALT1, IC19 LM317L, IC2 LM317L, IC20 A4983ALT1, IC21 LM317L, IC22 A4983ALT1, IC23 LM317L, IC24 A4983ALT1, IC25 LM317L, IC26 A4983ALT1, IC27 LM317L, IC28 A4983ALT1, IC29 LM317L, IC3 LM317L, IC30 A4983ALT1, IC31 LM317L, IC32 A4983ALT1, IC33 LM317L, IC34 A4983ALT1, IC35 LM317L, IC36 A4983ALT1, IC37 LM317L, IC38 A4983ALT1, IC39 LM317L, IC4 A4983ALT1, IC40 A4983ALT1, IC41 LM317L, IC42 A4983ALT1, IC43 LM317L, IC44 A4983ALT1, IC45 LM317L, IC46 A4983ALT1, IC47 LM317L, IC48 A4983ALT1, IC49 LM317L, IC5 LM317L, IC50 A4983ALT1, IC51 LM317L, IC52 A4983ALT1, IC53 LM317L, IC54 A4983ALT1, IC55 LM317L, IC56 A4983ALT1, IC57 LM317L, IC58 A4983ALT1, IC59 LM317L, IC6 A4983ALT1, IC60 A4983ALT1, IC61 LM317L, IC62 A4983ALT1, IC63 LM317L, IC64 A4983ALT1, IC65 LM317L, IC66 A4983ALT1, IC67 LM317L, IC68 A4983ALT1, IC69 LM317L, IC7 LM317L, IC70 A4983ALT1, IC71 LM317L, IC72 A4983ALT1, IC73 LM317L, IC74 A4983ALT1, IC75 LM317L, IC76 A4983ALT1, IC77 LM317L, IC78 A4983ALT1, IC79 LM317L, IC8 A4983ALT1, IC80 A4983ALT1, IC9 LM317L

Commit message: created panels v16a
Parts:
- removed 3/5V32, 3/5V33, 3/5V34, 3/5V35, 3/5V36, 3/5V37, 3/5V38, 3/5V39: SOLDERJUMPERNO, SparkFun03_30_09:SJ_2S-NO
- removed APWR32, APWR33, APWR34, APWR35, APWR36, APWR37, APWR38, APWR39: SOLDERJUMPERTRACE, SparkFun03_30_09:SJ_2S-TRACE
- removed C289, C298, C307, C316, C325, C334, C343, C352: .1uF, SparkFun-Capacitors:0603-CAP
- removed C290, C291, C292, C293, C295, C299, C300, C301, C302, C304, C308, C309, C310, C311, C313, C317, C318, C319, C320, C322, C326, C327, C328, C329, C331, C335, C336, C337, C338, C340, C344, C345, C346, C347, C349, C353, C354, C355, C356, C358: .1uf, SparkFun-Capacitors:0603-CAP
- removed C294, C303, C312, C321, C330, C339, C348, C357: .22uF, SparkFun-Capacitors:0603-CAP
- removed C296, C305, C314, C323, C332, C341, C350, C359: 47uF, SparkFun-Capacitors:PANASONIC_D
- removed C297, C306, C315, C324, C333, C342, C351, C360: 1uF, SparkFun-Capacitors:0603-CAP
- removed D33, D34, D35, D36, D37, D38, D39, D40: B340A-13-F, diode:DO-214AC
- removed E$5: (no value), SparkFun-Retired:FIDUCIAL-1.5X3
- removed FID65, FID66, FID67, FID68, FID69, FID70, FID71, FID72, FID73, FID74, FID75, FID76, FID77, FID78, FID79, FID80: FIDUCIAL1X2, SparkFun-Aesthetics:FIDUCIAL-1X2
- removed IC65, IC67, IC69, IC71, IC73, IC75, IC77, IC79: LM317L, BigEasyDriver_v11:SCHMALZHAUS_SOT89
- removed IC66, IC68, IC70, IC72, IC74, IC76, IC78, IC80: A4983ALT1, Testing:QFN-28-5MM_ALT1
- removed JP385, JP386, JP397, JP398, JP409, JP410, JP421, JP422, JP433, JP434, JP445, JP446, JP457, JP458, JP469, JP470: STAND-OFF, SparkFun-7-28-09:STAND-OFF
- removed JP387, JP389, JP399, JP401, JP411, JP413, JP423, JP425, JP435, JP437, JP447, JP449, JP459, JP461, JP471, JP473: (no value), SparkFun:1X02
- removed JP388, JP390, JP396, JP400, JP402, JP408, JP412, JP414, JP420, JP424, JP426, JP432, JP436, JP438, JP444, JP448, JP450, JP456, JP460, JP462, JP468, JP472, JP474, JP480: (no value), SparkFun:1X04
- removed JP391, JP393, JP394, JP403, JP405, JP406, JP415, JP417, JP418, JP427, JP429, JP430, JP439, JP441, JP442, JP451, JP453, JP454, JP463, JP465, JP466, JP475, JP477, JP478: (no value), BigEasyDriver_v11:SCREWTERMINAL-3.5MM-4_LOCK
- removed JP392, JP395, JP404, JP407, JP416, JP419, JP428, JP431, JP440, JP443, JP452, JP455, JP464, JP467, JP476, JP479: (no value), BigEasyDriver_v11:SCREWTERMINAL-3.5MM-2_LOCK
- removed LOGO33, LOGO34, LOGO35, LOGO36, LOGO37, LOGO38, LOGO39, LOGO40: OSHW_LOGO_FILLX0100-NT, OSHW:OSHW_FILLX100_NOTEXT
- removed PWR_LED32, PWR_LED33, PWR_LED34, PWR_LED35, PWR_LED36, PWR_LED37, PWR_LED38, PWR_LED39: YELLOW, SparkFun03_30_09:LED-0603
- removed R609, R628, R647, R666, R685, R704, R723, R742: 390, SparkFun-Resistors:0603-RES
- removed R610, R629, R648, R667, R686, R705, R724, R743: 240, SparkFun-Resistors:0603-RES
- removed R611, R626, R627, R630, R645, R646, R649, R664, R665, R668, R683, R684, R687, R702, R703, R706, R721, R722, R725, R740, R741, R744, R759, R760: 1K, SparkFun-Resistors:0603-RES
- removed R612, R631, R650, R669, R688, R707, R726, R745: 330, SparkFun-Resistors:0603-RES
- removed R613, R632, R651, R670, R689, R708, R727, R746: 10K, SparkFun-Electromechanical:TRIMPOT-3MM-2
- removed R614, R615, R633, R634, R652, R653, R671, R672, R690, R691, R709, R710, R728, R729, R747, R748: .11, SparkFun-Resistors:R2010
- removed R616, R617, R618, R619, R620, R621, R622, R623, R624, R635, R636, R637, R638, R639, R640, R641, R642, R643, R654, R655, R656, R657, R658, R659, R660, R661, R662, R673, R674, R675, R676, R677, R678, R679, R680, R681, R692, R693, R694, R695, R696, R697, R698, R699, R700, R711, R712, R713, R714, R715, R716, R717, R718, R719, R730, R731, R732, R733, R734, R735, R736, R737, R738, R749, R750, R751, R752, R753, R754, R755, R756, R757: 20K, SparkFun-Resistors:0603-RES
- removed R625, R644, R663, R682, R701, R720, R739, R758: 8.2K, SparkFun-Resistors:0603-RES
- removed TP33, TP34, TP35, TP36, TP37, TP38, TP39, TP40: TPPAD1-13, testpad:P1-13
- removed U$161, U$166, U$171, U$176, U$181, U$186, U$191, U$196: (no value), SchmalzHaus:SCHMALZHAUS_SMALL
- removed U$162, U$167, U$172, U$177, U$182, U$187, U$192, U$197: LOGO-SFENEW, SparkFun:SFE-NEW-WEBLOGO
- removed U$163, U$164, U$165, U$168, U$169, U$170, U$173, U$174, U$175, U$178, U$179, U$180, U$183, U$184, U$185, U$188, U$189, U$190, U$193, U$194, U$195, U$198, U$199, U$200: PAD, Testing:PAD-0.008
- added E$7: (no value), SparkFun-Aesthetics:FIDUCIAL-1X2
- E$4: device SparkFun-Aesthetics:FIDUCIAL-1X2 -> SparkFun-Retired:FIDUCIAL-1.5X3
- moved IC38 204.8 mm to (261.1, 22.1)
- moved IC39 204.8 mm to (285.4, 33.9)
- moved JP220 204.8 mm to (257.3, 32.3)
- moved JP222 204.8 mm to (257.3, 11.9)
- moved LOGO20 204.8 mm to (282.9, 13.4)
- moved R345 204.8 mm to (275.5, 15.9)
- moved R347 204.8 mm to (271.7, 19.8)
- moved R350 204.8 mm to (262.6, 15.9)
- moved U$95 204.8 mm to (261.1, 25.1)
- moved 3/5V16 204.8 mm to (172.5, 27.2)
- moved 3/5V17 204.8 mm to (209.8, 27.2)
- moved 3/5V18 204.8 mm to (247.1, 27.2)
- moved 3/5V19 204.8 mm to (284.5, 27.2)
- moved APWR16 204.8 mm to (175.0, 27.2)
- moved APWR17 204.8 mm to (212.3, 27.2)
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Connections:
- removed net 5V_ALT32: APWR32.1, IC65.OUT, IC65.OUT@1, R610.2
- removed net 5V_ALT33: APWR33.1, IC67.OUT, IC67.OUT@1, R629.2
- removed net 5V_ALT34: APWR34.1, IC69.OUT, IC69.OUT@1, R648.2
- removed net 5V_ALT35: APWR35.1, IC71.OUT, IC71.OUT@1, R667.2
- removed net 5V_ALT36: APWR36.1, IC73.OUT, IC73.OUT@1, R686.2
- removed net 5V_ALT37: APWR37.1, IC75.OUT, IC75.OUT@1, R705.2
- removed net 5V_ALT38: APWR38.1, IC77.OUT, IC77.OUT@1, R724.2
- removed net 5V_ALT39: APWR39.1, IC79.OUT, IC79.OUT@1, R743.2
- removed net COILA+32: IC66.P$21, JP388.4, JP391.4
- removed net COILA+33: IC68.P$21, JP400.4, JP403.4
- removed net COILA+34: IC70.P$21, JP412.4, JP415.4
- removed net COILA+35: IC72.P$21, JP424.4, JP427.4
- removed net COILA+36: IC74.P$21, JP436.4, JP439.4
- removed net COILA+37: IC76.P$21, JP448.4, JP451.4
- removed net COILA+38: IC78.P$21, JP460.4, JP463.4
- removed net COILA+39: IC80.P$21, JP472.4, JP475.4
- removed net COILA-32: IC66.P$24, JP388.3, JP391.3
- removed net COILA-33: IC68.P$24, JP400.3, JP403.3
- removed net COILA-34: IC70.P$24, JP412.3, JP415.3
- removed net COILA-35: IC72.P$24, JP424.3, JP427.3
- removed net COILA-36: IC74.P$24, JP436.3, JP439.3
- removed net COILA-37: IC76.P$24, JP448.3, JP451.3
- removed net COILA-38: IC78.P$24, JP460.3, JP463.3
- removed net COILA-39: IC80.P$24, JP472.3, JP475.3
- removed net COILB+32: IC66.P$1, JP388.1, JP391.1
- removed net COILB+33: IC68.P$1, JP400.1, JP403.1
- removed net COILB+34: IC70.P$1, JP412.1, JP415.1
- removed net COILB+35: IC72.P$1, JP424.1, JP427.1
- removed net COILB+36: IC74.P$1, JP436.1, JP439.1
- removed net COILB+37: IC76.P$1, JP448.1, JP451.1
- removed net COILB+38: IC78.P$1, JP460.1, JP463.1
- removed net COILB+39: IC80.P$1, JP472.1, JP475.1
- removed net COILB-32: IC66.P$26, JP388.2, JP391.2
- removed net COILB-33: IC68.P$26, JP400.2, JP403.2
- removed net COILB-34: IC70.P$26, JP412.2, JP415.2
- removed net COILB-35: IC72.P$26, JP424.2, JP427.2
- removed net COILB-36: IC74.P$26, JP436.2, JP439.2
- removed net COILB-37: IC76.P$26, JP448.2, JP451.2
- removed net COILB-38: IC78.P$26, JP460.2, JP463.2
- removed net COILB-39: IC80.P$26, JP472.2, JP475.2
- removed net CUR_REF32: IC66.P$17, R613.2, TP33.TP
- removed net CUR_REF33: IC68.P$17, R632.2, TP34.TP
- removed net CUR_REF34: IC70.P$17, R651.2, TP35.TP
- removed net CUR_REF35: IC72.P$17, R670.2, TP36.TP
- removed net CUR_REF36: IC74.P$17, R689.2, TP37.TP
- removed net CUR_REF37: IC76.P$17, R708.2, TP38.TP
- removed net CUR_REF38: IC78.P$17, R727.2, TP39.TP
- removed net CUR_REF39: IC80.P$17, R746.2, TP40.TP
- removed net DIR32: IC66.P$19, R623.1, R626.2
- removed net DIR33: IC68.P$19, R642.1, R645.2
- removed net DIR34: IC70.P$19, R661.1, R664.2
- removed net DIR35: IC72.P$19, R680.1, R683.2
- removed net DIR36: IC74.P$19, R699.1, R702.2
- removed net DIR37: IC76.P$19, R718.1, R721.2
- removed net DIR38: IC78.P$19, R737.1, R740.2
- removed net DIR39: IC80.P$19, R756.1, R759.2
- removed net DIR_IN32: JP394.4, JP396.4, R626.1
- removed net DIR_IN33: JP406.4, JP408.4, R645.1
- removed net DIR_IN34: JP418.4, JP420.4, R664.1
- removed net DIR_IN35: JP430.4, JP432.4, R683.1
- removed net DIR_IN36: JP442.4, JP444.4, R702.1
- removed net DIR_IN37: JP454.4, JP456.4, R721.1
- removed net DIR_IN38: JP466.4, JP468.4, R740.1
- removed net DIR_IN39: JP478.4, JP480.4, R759.1
- removed net ENABLE32: IC66.P$2, JP387.1, JP395.1, R622.1
- removed net ENABLE33: IC68.P$2, JP399.1, JP407.1, R641.1
- removed net ENABLE34: IC70.P$2, JP411.1, JP419.1, R660.1
- removed net ENABLE35: IC72.P$2, JP423.1, JP431.1, R679.1
- removed net ENABLE36: IC74.P$2, JP435.1, JP443.1, R698.1
- removed net ENABLE37: IC76.P$2, JP447.1, JP455.1, R717.1
- removed net ENABLE38: IC78.P$2, JP459.1, JP467.1, R736.1
- removed net ENABLE39: IC80.P$2, JP471.1, JP479.1, R755.1
- removed net GND32: 3/5V32.2, C289.2, C291.2, C292.2, C293.2, C294.2, C296.-, C297.2, IC66.P$18, IC66.P$29, IC66.P$3, JP389.1, JP392.1, JP394.2, JP396.2, PWR_LED32.C, R612.1, R613.3, R614.1, R615.1, R616.2, R622.2
- removed net GND33: 3/5V33.2, C298.2, C300.2, C301.2, C302.2, C303.2, C305.-, C306.2, IC68.P$18, IC68.P$29, IC68.P$3, JP401.1, JP404.1, JP406.2, JP408.2, PWR_LED33.C, R631.1, R632.3, R633.1, R634.1, R635.2, R641.2
- removed net GND34: 3/5V34.2, C307.2, C309.2, C310.2, C311.2, C312.2, C314.-, C315.2, IC70.P$18, IC70.P$29, IC70.P$3, JP413.1, JP416.1, JP418.2, JP420.2, PWR_LED34.C, R650.1, R651.3, R652.1, R653.1, R654.2, R660.2
- removed net GND35: 3/5V35.2, C316.2, C318.2, C319.2, C320.2, C321.2, C323.-, C324.2, IC72.P$18, IC72.P$29, IC72.P$3, JP425.1, JP428.1, JP430.2, JP432.2, PWR_LED35.C, R669.1, R670.3, R671.1, R672.1, R673.2, R679.2
- removed net GND36: 3/5V36.2, C325.2, C327.2, C328.2, C329.2, C330.2, C332.-, C333.2, IC74.P$18, IC74.P$29, IC74.P$3, JP437.1, JP440.1, JP442.2, JP444.2, PWR_LED36.C, R688.1, R689.3, R690.1, R691.1, R692.2, R698.2
- removed net GND37: 3/5V37.2, C334.2, C336.2, C337.2, C338.2, C339.2, C341.-, C342.2, IC76.P$18, IC76.P$29, IC76.P$3, JP449.1, JP452.1, JP454.2, JP456.2, PWR_LED37.C, R707.1, R708.3, R709.1, R710.1, R711.2, R717.2
- removed net GND38: 3/5V38.2, C343.2, C345.2, C346.2, C347.2, C348.2, C350.-, C351.2, IC78.P$18, IC78.P$29, IC78.P$3, JP461.1, JP464.1, JP466.2, JP468.2, PWR_LED38.C, R726.1, R727.3, R728.1, R729.1, R730.2, R736.2
- removed net GND39: 3/5V39.2, C352.2, C354.2, C355.2, C356.2, C357.2, C359.-, C360.2, IC80.P$18, IC80.P$29, IC80.P$3, JP473.1, JP476.1, JP478.2, JP480.2, PWR_LED39.C, R745.1, R746.3, R747.1, R748.1, R749.2, R755.2
- removed net MS100: IC68.P$9, JP399.2, JP407.2, R636.1
- removed net MS101: IC68.P$10, JP402.1, JP405.1, R637.1
- removed net MS102: IC68.P$11, JP402.2, JP405.2, R638.1
- removed net MS103: IC70.P$9, JP411.2, JP419.2, R655.1
- removed net MS104: IC70.P$10, JP414.1, JP417.1, R656.1
- removed net MS105: IC70.P$11, JP414.2, JP417.2, R657.1
- removed net MS106: IC72.P$9, JP423.2, JP431.2, R674.1
- removed net MS107: IC72.P$10, JP426.1, JP429.1, R675.1
- removed net MS108: IC72.P$11, JP426.2, JP429.2, R676.1
- removed net MS109: IC74.P$9, JP435.2, JP443.2, R693.1
- removed net MS110: IC74.P$10, JP438.1, JP441.1, R694.1
- removed net MS111: IC74.P$11, JP438.2, JP441.2, R695.1
- removed net MS112: IC76.P$9, JP447.2, JP455.2, R712.1
- removed net MS113: IC76.P$10, JP450.1, JP453.1, R713.1
- removed net MS114: IC76.P$11, JP450.2, JP453.2, R714.1
- removed net MS115: IC78.P$9, JP459.2, JP467.2, R731.1
- removed net MS116: IC78.P$10, JP462.1, JP465.1, R732.1
- removed net MS117: IC78.P$11, JP462.2, JP465.2, R733.1
- removed net MS118: IC80.P$9, JP471.2, JP479.2, R750.1
- removed net MS119: IC80.P$10, JP474.1, JP477.1, R751.1
- removed net MS120: IC80.P$11, JP474.2, JP477.2, R752.1
- removed net MS97: IC66.P$9, JP387.2, JP395.2, R617.1
- removed net MS98: IC66.P$10, JP390.1, JP393.1, R618.1
- removed net MS99: IC66.P$11, JP390.2, JP393.2, R619.1
- removed net N$481: IC65.ADJ, R609.2, R610.1
- removed net N$482: PWR_LED32.A, R611.1
- removed net N$483: 3/5V32.1, R609.1, R612.2
- removed net N$484: IC66.P$27, R614.2
- removed net N$485: IC66.P$23, R615.2
- removed net N$486: C290.1, IC66.P$4
- removed net N$487: C290.2, IC66.P$5
- removed net N$488: IC66.P$13, R616.1
- removed net N$489: C294.1, IC66.P$8
- removed net N$490: C295.1, IC66.P$6
- removed net N$491: D33.A, JP389.2, JP392.2
- removed net N$492: R613.1, R625.2
- removed net N$493: IC66.P$7, U$163.P$1
- removed net N$494: IC66.P$20, U$164.P$1
- removed net N$495: IC66.P$25, U$165.P$1
- removed net N$496: IC67.ADJ, R628.2, R629.1
- removed net N$497: PWR_LED33.A, R630.1
- removed net N$498: 3/5V33.1, R628.1, R631.2
- removed net N$499: IC68.P$27, R633.2
- removed net N$500: IC68.P$23, R634.2
- removed net N$501: C299.1, IC68.P$4
- removed net N$502: C299.2, IC68.P$5
- removed net N$503: IC68.P$13, R635.1
- removed net N$504: C303.1, IC68.P$8
- removed net N$505: C304.1, IC68.P$6
- removed net N$506: D34.A, JP401.2, JP404.2
- removed net N$507: R632.1, R644.2
- removed net N$508: IC68.P$7, U$168.P$1
- removed net N$509: IC68.P$20, U$169.P$1
- removed net N$510: IC68.P$25, U$170.P$1
- removed net N$511: IC69.ADJ, R647.2, R648.1
- removed net N$512: PWR_LED34.A, R649.1
- removed net N$513: 3/5V34.1, R647.1, R650.2
- removed net N$514: IC70.P$27, R652.2
- removed net N$515: IC70.P$23, R653.2
- removed net N$516: C308.1, IC70.P$4
- removed net N$517: C308.2, IC70.P$5
- removed net N$518: IC70.P$13, R654.1
- removed net N$519: C312.1, IC70.P$8
- removed net N$520: C313.1, IC70.P$6
- removed net N$521: D35.A, JP413.2, JP416.2
- removed net N$522: R651.1, R663.2
- removed net N$523: IC70.P$7, U$173.P$1
- removed net N$524: IC70.P$20, U$174.P$1
- removed net N$525: IC70.P$25, U$175.P$1
- removed net N$526: IC71.ADJ, R666.2, R667.1
- removed net N$527: PWR_LED35.A, R668.1
- removed net N$528: 3/5V35.1, R666.1, R669.2
- removed net N$529: IC72.P$27, R671.2
- removed net N$530: IC72.P$23, R672.2
- removed net N$531: C317.1, IC72.P$4
- removed net N$532: C317.2, IC72.P$5
- removed net N$533: IC72.P$13, R673.1
- removed net N$534: C321.1, IC72.P$8
- removed net N$535: C322.1, IC72.P$6
- removed net N$536: D36.A, JP425.2, JP428.2
- removed net N$537: R670.1, R682.2
- removed net N$538: IC72.P$7, U$178.P$1
- removed net N$539: IC72.P$20, U$179.P$1
- removed net N$540: IC72.P$25, U$180.P$1
- removed net N$541: IC73.ADJ, R685.2, R686.1
- removed net N$542: PWR_LED36.A, R687.1
- removed net N$543: 3/5V36.1, R685.1, R688.2
- removed net N$544: IC74.P$27, R690.2
- removed net N$545: IC74.P$23, R691.2
- removed net N$546: C326.1, IC74.P$4
- removed net N$547: C326.2, IC74.P$5
- removed net N$548: IC74.P$13, R692.1
- removed net N$549: C330.1, IC74.P$8
- removed net N$550: C331.1, IC74.P$6
- removed net N$551: D37.A, JP437.2, JP440.2
- removed net N$552: R689.1, R701.2
- removed net N$553: IC74.P$7, U$183.P$1
- removed net N$554: IC74.P$20, U$184.P$1
- removed net N$555: IC74.P$25, U$185.P$1
- removed net N$556: IC75.ADJ, R704.2, R705.1
- removed net N$557: PWR_LED37.A, R706.1
- removed net N$558: 3/5V37.1, R704.1, R707.2
- removed net N$559: IC76.P$27, R709.2
- removed net N$560: IC76.P$23, R710.2
- removed net N$561: C335.1, IC76.P$4
- removed net N$562: C335.2, IC76.P$5
- removed net N$563: IC76.P$13, R711.1
- removed net N$564: C339.1, IC76.P$8
- removed net N$565: C340.1, IC76.P$6
- removed net N$566: D38.A, JP449.2, JP452.2
- removed net N$567: R708.1, R720.2
- removed net N$568: IC76.P$7, U$188.P$1
- removed net N$569: IC76.P$20, U$189.P$1
- removed net N$570: IC76.P$25, U$190.P$1
- removed net N$571: IC77.ADJ, R723.2, R724.1
- removed net N$572: PWR_LED38.A, R725.1
- removed net N$573: 3/5V38.1, R723.1, R726.2
- removed net N$574: IC78.P$27, R728.2
- removed net N$575: IC78.P$23, R729.2
- removed net N$576: C344.1, IC78.P$4
- removed net N$577: C344.2, IC78.P$5
- removed net N$578: IC78.P$13, R730.1
- removed net N$579: C348.1, IC78.P$8
- removed net N$580: C349.1, IC78.P$6
- removed net N$581: D39.A, JP461.2, JP464.2
- removed net N$582: R727.1, R739.2
- removed net N$583: IC78.P$7, U$193.P$1
- removed net N$584: IC78.P$20, U$194.P$1
- removed net N$585: IC78.P$25, U$195.P$1
- removed net N$586: IC79.ADJ, R742.2, R743.1
- removed net N$587: PWR_LED39.A, R744.1
- removed net N$588: 3/5V39.1, R742.1, R745.2
- removed net N$589: IC80.P$27, R747.2
- removed net N$590: IC80.P$23, R748.2
- removed net N$591: C353.1, IC80.P$4
- removed net N$592: C353.2, IC80.P$5
- removed net N$593: IC80.P$13, R749.1
- removed net N$594: C357.1, IC80.P$8
- removed net N$595: C358.1, IC80.P$6
- removed net N$596: D40.A, JP473.2, JP476.2
- removed net N$597: R746.1, R758.2
- removed net N$598: IC80.P$7, U$198.P$1
- removed net N$599: IC80.P$20, U$199.P$1
- removed net N$600: IC80.P$25, U$200.P$1
- removed net RESET32: IC66.P$12, JP390.3, JP393.3, R621.1
- removed net RESET33: IC68.P$12, JP402.3, JP405.3, R640.1
- removed net RESET34: IC70.P$12, JP414.3, JP417.3, R659.1
- removed net RESET35: IC72.P$12, JP426.3, JP429.3, R678.1
- removed net RESET36: IC74.P$12, JP438.3, JP441.3, R697.1
- removed net RESET37: IC76.P$12, JP450.3, JP453.3, R716.1
- removed net RESET38: IC78.P$12, JP462.3, JP465.3, R735.1
- removed net RESET39: IC80.P$12, JP474.3, JP477.3, R754.1
- removed net SLEEP32: IC66.P$14, JP390.4, JP393.4, R620.1
- removed net SLEEP33: IC68.P$14, JP402.4, JP405.4, R639.1
- removed net SLEEP34: IC70.P$14, JP414.4, JP417.4, R658.1
- removed net SLEEP35: IC72.P$14, JP426.4, JP429.4, R677.1
- removed net SLEEP36: IC74.P$14, JP438.4, JP441.4, R696.1
- removed net SLEEP37: IC76.P$14, JP450.4, JP453.4, R715.1
- removed net SLEEP38: IC78.P$14, JP462.4, JP465.4, R734.1
- removed net SLEEP39: IC80.P$14, JP474.4, JP477.4, R753.1
- removed net STEP32: IC66.P$16, R624.1, R627.2
- removed net STEP33: IC68.P$16, R643.1, R646.2
- removed net STEP34: IC70.P$16, R662.1, R665.2
- removed net STEP35: IC72.P$16, R681.1, R684.2
- removed net STEP36: IC74.P$16, R700.1, R703.2
- removed net STEP37: IC76.P$16, R719.1, R722.2
- removed net STEP38: IC78.P$16, R738.1, R741.2
- removed net STEP39: IC80.P$16, R757.1, R760.2
- removed net STEP_IN32: JP394.3, JP396.3, R627.1
- removed net STEP_IN33: JP406.3, JP408.3, R646.1
- removed net STEP_IN34: JP418.3, JP420.3, R665.1
- removed net STEP_IN35: JP430.3, JP432.3, R684.1
- removed net STEP_IN36: JP442.3, JP444.3, R703.1
- removed net STEP_IN37: JP454.3, JP456.3, R722.1
- removed net STEP_IN38: JP466.3, JP468.3, R741.1
- removed net STEP_IN39: JP478.3, JP480.3, R760.1
- removed net V+32: C289.1, C292.1, C293.1, C295.2, C296.+, D33.C, IC65.IN, IC66.P$22, IC66.P$28
- removed net V+33: C298.1, C301.1, C302.1, C304.2, C305.+, D34.C, IC67.IN, IC68.P$22, IC68.P$28
- removed net V+34: C307.1, C310.1, C311.1, C313.2, C314.+, D35.C, IC69.IN, IC70.P$22, IC70.P$28
- removed net V+35: C316.1, C319.1, C320.1, C322.2, C323.+, D36.C, IC71.IN, IC72.P$22, IC72.P$28
- removed net V+36: C325.1, C328.1, C329.1, C331.2, C332.+, D37.C, IC73.IN, IC74.P$22, IC74.P$28
- removed net V+37: C334.1, C337.1, C338.1, C340.2, C341.+, D38.C, IC75.IN, IC76.P$22, IC76.P$28
- removed net V+38: C343.1, C346.1, C347.1, C349.2, C350.+, D39.C, IC77.IN, IC78.P$22, IC78.P$28
- removed net V+39: C352.1, C355.1, C356.1, C358.2, C359.+, D40.C, IC79.IN, IC80.P$22, IC80.P$28
- removed net VCC32: APWR32.2, C291.1, C297.1, IC66.P$15, JP394.1, JP396.1, R611.2, R617.2, R618.2, R619.2, R620.2, R621.2, R623.2, R624.2, R625.1
- removed net VCC33: APWR33.2, C300.1, C306.1, IC68.P$15, JP406.1, JP408.1, R630.2, R636.2, R637.2, R638.2, R639.2, R640.2, R642.2, R643.2, R644.1
- removed net VCC34: APWR34.2, C309.1, C315.1, IC70.P$15, JP418.1, JP420.1, R649.2, R655.2, R656.2, R657.2, R658.2, R659.2, R661.2, R662.2, R663.1
- removed net VCC35: APWR35.2, C318.1, C324.1, IC72.P$15, JP430.1, JP432.1, R668.2, R674.2, R675.2, R676.2, R677.2, R678.2, R680.2, R681.2, R682.1
- removed net VCC36: APWR36.2, C327.1, C333.1, IC74.P$15, JP442.1, JP444.1, R687.2, R693.2, R694.2, R695.2, R696.2, R697.2, R699.2, R700.2, R701.1
- removed net VCC37: APWR37.2, C336.1, C342.1, IC76.P$15, JP454.1, JP456.1, R706.2, R712.2, R713.2, R714.2, R715.2, R716.2, R718.2, R719.2, R720.1
- removed net VCC38: APWR38.2, C345.1, C351.1, IC78.P$15, JP466.1, JP468.1, R725.2, R731.2, R732.2, R733.2, R734.2, R735.2, R737.2, R738.2, R739.1
- removed net VCC39: APWR39.2, C354.1, C360.1, IC80.P$15, JP478.1, JP480.1, R744.2, R750.2, R751.2, R752.2, R753.2, R754.2, R756.2, R757.2, R758.1
Routing:
- net V+33: track 58.8 -> 0.00 mm, vias 6 -> 0
- net V+32: track 58.8 -> 0.00 mm, vias 6 -> 0
- net V+37: track 58.8 -> 0.00 mm, vias 6 -> 0
- net V+34: track 58.8 -> 0.00 mm, vias 6 -> 0
- net V+35: track 58.8 -> 0.00 mm, vias 6 -> 0
- net V+36: track 58.8 -> 0.00 mm, vias 6 -> 0
- net V+38: track 58.8 -> 0.00 mm, vias 6 -> 0
- net V+39: track 58.8 -> 0.00 mm, vias 6 -> 0
- net VCC38: track 34.8 -> 0.00 mm, vias 3 -> 0
- net VCC34: track 34.8 -> 0.00 mm, vias 3 -> 0
- net VCC33: track 34.8 -> 0.00 mm, vias 3 -> 0
- net VCC37: track 34.8 -> 0.00 mm, vias 3 -> 0
- net VCC36: track 34.8 -> 0.00 mm, vias 3 -> 0
- net VCC32: track 34.8 -> 0.00 mm, vias 3 -> 0
- net VCC39: track 34.8 -> 0.00 mm, vias 3 -> 0
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- removed copper zone on layer 1, net 5V_ALT32
- removed copper zone on layer 1, net 5V_ALT33
- removed copper zone on layer 1, net 5V_ALT34
- removed copper zone on layer 1, net 5V_ALT35
- removed copper zone on layer 1, net 5V_ALT36
- removed copper zone on layer 1, net 5V_ALT37
- removed copper zone on layer 1, net 5V_ALT38
- removed copper zone on layer 1, net 5V_ALT39
- removed copper zone on layer 1, net COILA+32
- removed copper zone on layer 16, net COILA+32
- removed copper zone on layer 1, net COILA+33
- removed copper zone on layer 16, net COILA+33
- removed copper zone on layer 1, net COILA+34
- removed copper zone on layer 16, net COILA+34
- removed copper zone on layer 1, net COILA+35
- removed copper zone on layer 16, net COILA+35
- removed copper zone on layer 1, net COILA+36
- removed copper zone on layer 16, net COILA+36
- removed copper zone on layer 1, net COILA+37
- removed copper zone on layer 16, net COILA+37
- removed copper zone on layer 1, net COILA+38
- removed copper zone on layer 16, net COILA+38
- removed copper zone on layer 1, net COILA+39
- removed copper zone on layer 16, net COILA+39
- removed copper zone on layer 1, net COILA-32
- removed copper zone on layer 1, net COILA-33
- removed copper zone on layer 1, net COILA-34
- removed copper zone on layer 1, net COILA-35
- removed copper zone on layer 1, net COILA-36
- removed copper zone on layer 1, net COILA-37
- removed copper zone on layer 1, net COILA-38
- removed copper zone on layer 1, net COILA-39
- removed copper zone on layer 1, net COILB+32
- removed copper zone on layer 16, net COILB+32
- removed copper zone on layer 1, net COILB+33
- removed copper zone on layer 16, net COILB+33
- removed copper zone on layer 1, net COILB+34
- removed copper zone on layer 16, net COILB+34
- removed copper zone on layer 1, net COILB+35
- removed copper zone on layer 16, net COILB+35
- removed copper zone on layer 1, net COILB+36
- removed copper zone on layer 16, net COILB+36
- removed copper zone on layer 1, net COILB+37
- removed copper zone on layer 16, net COILB+37
- removed copper zone on layer 1, net COILB+38
- removed copper zone on layer 16, net COILB+38
- removed copper zone on layer 1, net COILB+39
- removed copper zone on layer 16, net COILB+39
- removed copper zone on layer 1, net COILB-32
- removed copper zone on layer 1, net COILB-33
- removed copper zone on layer 1, net COILB-34
- removed copper zone on layer 1, net COILB-35
- removed copper zone on layer 1, net COILB-36
- removed copper zone on layer 1, net COILB-37
- removed copper zone on layer 1, net COILB-38
- removed copper zone on layer 1, net COILB-39
- removed copper zone on layer 1, net GND32
- removed copper zone on layer 15, net GND32
- removed copper zone on layer 16, net GND32
- removed copper zone on layer 1, net GND33
- removed copper zone on layer 15, net GND33
- removed copper zone on layer 16, net GND33
- removed copper zone on layer 1, net GND34
- removed copper zone on layer 15, net GND34
- removed copper zone on layer 16, net GND34
- removed copper zone on layer 1, net GND35
- removed copper zone on layer 15, net GND35
- removed copper zone on layer 16, net GND35
- removed copper zone on layer 1, net GND36
- removed copper zone on layer 15, net GND36
- removed copper zone on layer 16, net GND36
- removed copper zone on layer 1, net GND37
- removed copper zone on layer 15, net GND37
- removed copper zone on layer 16, net GND37
- removed copper zone on layer 1, net GND38
- removed copper zone on layer 15, net GND38
- removed copper zone on layer 16, net GND38
- removed copper zone on layer 1, net GND39
- removed copper zone on layer 15, net GND39
- removed copper zone on layer 16, net GND39
- removed copper zone on layer 1, net N$484
- removed copper zone on layer 1, net N$485
- removed copper zone on layer 1, net N$499
- removed copper zone on layer 1, net N$500
- removed copper zone on layer 1, net N$514
- removed copper zone on layer 1, net N$515
- removed copper zone on layer 1, net N$529
- removed copper zone on layer 1, net N$530
- removed copper zone on layer 1, net N$544
- removed copper zone on layer 1, net N$545
- removed copper zone on layer 1, net N$559
- removed copper zone on layer 1, net N$560
- removed copper zone on layer 1, net N$574
- removed copper zone on layer 1, net N$575
- removed copper zone on layer 1, net N$589
- removed copper zone on layer 1, net N$590
- removed copper zone on layer 1, net V+32
- removed copper zone on layer 1, net V+33
- removed copper zone on layer 1, net V+34
- removed copper zone on layer 1, net V+35
- removed copper zone on layer 1, net V+36
- removed copper zone on layer 1, net V+37
- removed copper zone on layer 1, net V+38
- removed copper zone on layer 1, net V+39
- removed copper zone on layer 2, net VCC32
- removed copper zone on layer 2, net VCC33
- removed copper zone on layer 2, net VCC34
- removed copper zone on layer 2, net VCC35
- removed copper zone on layer 2, net VCC36
- removed copper zone on layer 2, net VCC37
- removed copper zone on layer 2, net VCC38
- removed copper zone on layer 2, net VCC39
Other:
- board size 325.6 x 168.1 mm -> 325.6 x 137.2 mm
- board text added: "v16a"
- board text removed: "This is a 4-layer board!!"
- board text removed: "v16"
