File: Production_Files/BigEasyDriver_Panel_v16a.brd (EAGLE design)
At the start: 162.6 x 168.1 mm, 1103 parts, among them IC1 A4983ALT1, IC10 A4983ALT1, IC11 LM317L, IC12 A4983ALT1, IC13 LM317L, IC14 A4983ALT1, IC15 LM317L, IC16 A4983ALT1, IC17 LM317L, IC18 A4983ALT1, IC19 LM317L, IC2 LM317L, IC20 A4983ALT1, IC21 LM317L, IC22 A4983ALT1, IC23 LM317L, IC24 A4983ALT1, IC25 LM317L, IC26 A4983ALT1, IC27 LM317L, IC28 A4983ALT1, IC29 LM317L, IC3 LM317L, IC30 A4983ALT1, IC31 LM317L, IC32 A4983ALT1, IC33 LM317L, IC34 A4983ALT1, IC35 LM317L, IC36 A4983ALT1, IC37 LM317L, IC38 A4983ALT1, IC39 LM317L, IC4 A4983ALT1, IC40 A4983ALT1, IC5 LM317L, IC6 A4983ALT1, IC7 LM317L, IC8 A4983ALT1, IC9 LM317L

Commit message: created panels v16a
Parts:
- removed 3/5V16, 3/5V17, 3/5V18, 3/5V19: SOLDERJUMPERNO, SparkFun03_30_09:SJ_2S-NO
- removed APWR16, APWR17, APWR18, APWR19: SOLDERJUMPERTRACE, SparkFun03_30_09:SJ_2S-TRACE
- removed C145, C154, C163, C172: .1uF, SparkFun-Capacitors:0603-CAP
- removed C146, C147, C148, C149, C151, C155, C156, C157, C158, C160, C164, C165, C166, C167, C169, C173, C174, C175, C176, C178: .1uf, SparkFun-Capacitors:0603-CAP
- removed C150, C159, C168, C177: .22uF, SparkFun-Capacitors:0603-CAP
- removed C152, C161, C170, C179: 47uF, SparkFun-Capacitors:PANASONIC_D
- removed C153, C162, C171, C180: 1uF, SparkFun-Capacitors:0603-CAP
- removed D17, D18, D19, D20: B340A-13-F, diode:DO-214AC
- removed E$4: (no value), SparkFun-Aesthetics:FIDUCIAL-1X2
- removed FID33, FID34, FID35, FID36, FID37, FID38, FID39, FID40: FIDUCIAL1X2, SparkFun-Aesthetics:FIDUCIAL-1X2
- removed IC33, IC35, IC37, IC39: LM317L, BigEasyDriver_v11:SCHMALZHAUS_SOT89
- removed IC34, IC36, IC38, IC40: A4983ALT1, Testing:QFN-28-5MM_ALT1
- removed JP193, JP194, JP205, JP206, JP217, JP218, JP229, JP230: STAND-OFF, SparkFun-7-28-09:STAND-OFF
- removed JP195, JP197, JP207, JP209, JP219, JP221, JP231, JP233: (no value), SparkFun:1X02
- removed JP196, JP198, JP204, JP208, JP210, JP216, JP220, JP222, JP228, JP232, JP234, JP240: (no value), SparkFun:1X04
- removed JP199, JP201, JP202, JP211, JP213, JP214, JP223, JP225, JP226, JP235, JP237, JP238: (no value), BigEasyDriver_v11:SCREWTERMINAL-3.5MM-4_LOCK
- removed JP200, JP203, JP212, JP215, JP224, JP227, JP236, JP239: (no value), BigEasyDriver_v11:SCREWTERMINAL-3.5MM-2_LOCK
- removed LOGO17, LOGO18, LOGO19, LOGO20: OSHW_LOGO_FILLX0100-NT, OSHW:OSHW_FILLX100_NOTEXT
- removed PWR_LED16, PWR_LED17, PWR_LED18, PWR_LED19: YELLOW, SparkFun03_30_09:LED-0603
- removed R305, R324, R343, R362: 390, SparkFun-Resistors:0603-RES
- removed R306, R325, R344, R363: 240, SparkFun-Resistors:0603-RES
- removed R307, R322, R323, R326, R341, R342, R345, R360, R361, R364, R379, R380: 1K, SparkFun-Resistors:0603-RES
- removed R308, R327, R346, R365: 330, SparkFun-Resistors:0603-RES
- removed R309, R328, R347, R366: 10K, SparkFun-Electromechanical:TRIMPOT-3MM-2
- removed R310, R311, R329, R330, R348, R349, R367, R368: .11, SparkFun-Resistors:R2010
- removed R312, R313, R314, R315, R316, R317, R318, R319, R320, R331, R332, R333, R334, R335, R336, R337, R338, R339, R350, R351, R352, R353, R354, R355, R356, R357, R358, R369, R370, R371, R372, R373, R374, R375, R376, R377: 20K, SparkFun-Resistors:0603-RES
- removed R321, R340, R359, R378: 8.2K, SparkFun-Resistors:0603-RES
- removed TP17, TP18, TP19, TP20: TPPAD1-13, testpad:P1-13
- removed U$100, U$83, U$84, U$85, U$88, U$89, U$90, U$93, U$94, U$95, U$98, U$99: PAD, Testing:PAD-0.008
- removed U$81, U$86, U$91, U$96: (no value), SchmalzHaus:SCHMALZHAUS_SMALL
- removed U$82, U$87, U$92, U$97: LOGO-SFENEW, SparkFun:SFE-NEW-WEBLOGO
- added E$7: (no value), SparkFun-Aesthetics:FIDUCIAL-1X2
- moved E$6 33.6 mm to (158.1, 124.0)
- moved E$1 3.56 mm to (4.57, 14.5)
Connections:
- removed net 5V_ALT16: APWR16.1, IC33.OUT, IC33.OUT@1, R306.2
- removed net 5V_ALT17: APWR17.1, IC35.OUT, IC35.OUT@1, R325.2
- removed net 5V_ALT18: APWR18.1, IC37.OUT, IC37.OUT@1, R344.2
- removed net 5V_ALT19: APWR19.1, IC39.OUT, IC39.OUT@1, R363.2
- removed net COILA+16: IC34.P$21, JP196.4, JP199.4
- removed net COILA+17: IC36.P$21, JP208.4, JP211.4
- removed net COILA+18: IC38.P$21, JP220.4, JP223.4
- removed net COILA+19: IC40.P$21, JP232.4, JP235.4
- removed net COILA-16: IC34.P$24, JP196.3, JP199.3
- removed net COILA-17: IC36.P$24, JP208.3, JP211.3
- removed net COILA-18: IC38.P$24, JP220.3, JP223.3
- removed net COILA-19: IC40.P$24, JP232.3, JP235.3
- removed net COILB+16: IC34.P$1, JP196.1, JP199.1
- removed net COILB+17: IC36.P$1, JP208.1, JP211.1
- removed net COILB+18: IC38.P$1, JP220.1, JP223.1
- removed net COILB+19: IC40.P$1, JP232.1, JP235.1
- removed net COILB-16: IC34.P$26, JP196.2, JP199.2
- removed net COILB-17: IC36.P$26, JP208.2, JP211.2
- removed net COILB-18: IC38.P$26, JP220.2, JP223.2
- removed net COILB-19: IC40.P$26, JP232.2, JP235.2
- removed net CUR_REF16: IC34.P$17, R309.2, TP17.TP
- removed net CUR_REF17: IC36.P$17, R328.2, TP18.TP
- removed net CUR_REF18: IC38.P$17, R347.2, TP19.TP
- removed net CUR_REF19: IC40.P$17, R366.2, TP20.TP
- removed net DIR16: IC34.P$19, R319.1, R322.2
- removed net DIR17: IC36.P$19, R338.1, R341.2
- removed net DIR18: IC38.P$19, R357.1, R360.2
- removed net DIR19: IC40.P$19, R376.1, R379.2
- removed net DIR_IN16: JP202.4, JP204.4, R322.1
- removed net DIR_IN17: JP214.4, JP216.4, R341.1
- removed net DIR_IN18: JP226.4, JP228.4, R360.1
- removed net DIR_IN19: JP238.4, JP240.4, R379.1
- removed net ENABLE16: IC34.P$2, JP195.1, JP203.1, R318.1
- removed net ENABLE17: IC36.P$2, JP207.1, JP215.1, R337.1
- removed net ENABLE18: IC38.P$2, JP219.1, JP227.1, R356.1
- removed net ENABLE19: IC40.P$2, JP231.1, JP239.1, R375.1
- removed net GND16: 3/5V16.2, C145.2, C147.2, C148.2, C149.2, C150.2, C152.-, C153.2, IC34.P$18, IC34.P$29, IC34.P$3, JP197.1, JP200.1, JP202.2, JP204.2, PWR_LED16.C, R308.1, R309.3, R310.1, R311.1, R312.2, R318.2
- removed net GND17: 3/5V17.2, C154.2, C156.2, C157.2, C158.2, C159.2, C161.-, C162.2, IC36.P$18, IC36.P$29, IC36.P$3, JP209.1, JP212.1, JP214.2, JP216.2, PWR_LED17.C, R327.1, R328.3, R329.1, R330.1, R331.2, R337.2
- removed net GND18: 3/5V18.2, C163.2, C165.2, C166.2, C167.2, C168.2, C170.-, C171.2, IC38.P$18, IC38.P$29, IC38.P$3, JP221.1, JP224.1, JP226.2, JP228.2, PWR_LED18.C, R346.1, R347.3, R348.1, R349.1, R350.2, R356.2
- removed net GND19: 3/5V19.2, C172.2, C174.2, C175.2, C176.2, C177.2, C179.-, C180.2, IC40.P$18, IC40.P$29, IC40.P$3, JP233.1, JP236.1, JP238.2, JP240.2, PWR_LED19.C, R365.1, R366.3, R367.1, R368.1, R369.2, R375.2
- removed net MS49: IC34.P$9, JP195.2, JP203.2, R313.1
- removed net MS50: IC34.P$10, JP198.1, JP201.1, R314.1
- removed net MS51: IC34.P$11, JP198.2, JP201.2, R315.1
- removed net MS52: IC36.P$9, JP207.2, JP215.2, R332.1
- removed net MS53: IC36.P$10, JP210.1, JP213.1, R333.1
- removed net MS54: IC36.P$11, JP210.2, JP213.2, R334.1
- removed net MS55: IC38.P$9, JP219.2, JP227.2, R351.1
- removed net MS56: IC38.P$10, JP222.1, JP225.1, R352.1
- removed net MS57: IC38.P$11, JP222.2, JP225.2, R353.1
- removed net MS58: IC40.P$9, JP231.2, JP239.2, R370.1
- removed net MS59: IC40.P$10, JP234.1, JP237.1, R371.1
- removed net MS60: IC40.P$11, JP234.2, JP237.2, R372.1
- removed net N$241: IC33.ADJ, R305.2, R306.1
- removed net N$242: PWR_LED16.A, R307.1
- removed net N$243: 3/5V16.1, R305.1, R308.2
- removed net N$244: IC34.P$27, R310.2
- removed net N$245: IC34.P$23, R311.2
- removed net N$246: C146.1, IC34.P$4
- removed net N$247: C146.2, IC34.P$5
- removed net N$248: IC34.P$13, R312.1
- removed net N$249: C150.1, IC34.P$8
- removed net N$250: C151.1, IC34.P$6
- removed net N$251: D17.A, JP197.2, JP200.2
- removed net N$252: R309.1, R321.2
- removed net N$253: IC34.P$7, U$83.P$1
- removed net N$254: IC34.P$20, U$84.P$1
- removed net N$255: IC34.P$25, U$85.P$1
- removed net N$256: IC35.ADJ, R324.2, R325.1
- removed net N$257: PWR_LED17.A, R326.1
- removed net N$258: 3/5V17.1, R324.1, R327.2
- removed net N$259: IC36.P$27, R329.2
- removed net N$260: IC36.P$23, R330.2
- removed net N$261: C155.1, IC36.P$4
- removed net N$262: C155.2, IC36.P$5
- removed net N$263: IC36.P$13, R331.1
- removed net N$264: C159.1, IC36.P$8
- removed net N$265: C160.1, IC36.P$6
- removed net N$266: D18.A, JP209.2, JP212.2
- removed net N$267: R328.1, R340.2
- removed net N$268: IC36.P$7, U$88.P$1
- removed net N$269: IC36.P$20, U$89.P$1
- removed net N$270: IC36.P$25, U$90.P$1
- removed net N$271: IC37.ADJ, R343.2, R344.1
- removed net N$272: PWR_LED18.A, R345.1
- removed net N$273: 3/5V18.1, R343.1, R346.2
- removed net N$274: IC38.P$27, R348.2
- removed net N$275: IC38.P$23, R349.2
- removed net N$276: C164.1, IC38.P$4
- removed net N$277: C164.2, IC38.P$5
- removed net N$278: IC38.P$13, R350.1
- removed net N$279: C168.1, IC38.P$8
- removed net N$280: C169.1, IC38.P$6
- removed net N$281: D19.A, JP221.2, JP224.2
- removed net N$282: R347.1, R359.2
- removed net N$283: IC38.P$7, U$93.P$1
- removed net N$284: IC38.P$20, U$94.P$1
- removed net N$285: IC38.P$25, U$95.P$1
- removed net N$286: IC39.ADJ, R362.2, R363.1
- removed net N$287: PWR_LED19.A, R364.1
- removed net N$288: 3/5V19.1, R362.1, R365.2
- removed net N$289: IC40.P$27, R367.2
- removed net N$290: IC40.P$23, R368.2
- removed net N$291: C173.1, IC40.P$4
- removed net N$292: C173.2, IC40.P$5
- removed net N$293: IC40.P$13, R369.1
- removed net N$294: C177.1, IC40.P$8
- removed net N$295: C178.1, IC40.P$6
- removed net N$296: D20.A, JP233.2, JP236.2
- removed net N$297: R366.1, R378.2
- removed net N$298: IC40.P$7, U$98.P$1
- removed net N$299: IC40.P$20, U$99.P$1
- removed net N$300: IC40.P$25, U$100.P$1
- removed net RESET16: IC34.P$12, JP198.3, JP201.3, R317.1
- removed net RESET17: IC36.P$12, JP210.3, JP213.3, R336.1
- removed net RESET18: IC38.P$12, JP222.3, JP225.3, R355.1
- removed net RESET19: IC40.P$12, JP234.3, JP237.3, R374.1
- removed net SLEEP16: IC34.P$14, JP198.4, JP201.4, R316.1
- removed net SLEEP17: IC36.P$14, JP210.4, JP213.4, R335.1
- removed net SLEEP18: IC38.P$14, JP222.4, JP225.4, R354.1
- removed net SLEEP19: IC40.P$14, JP234.4, JP237.4, R373.1
- removed net STEP16: IC34.P$16, R320.1, R323.2
- removed net STEP17: IC36.P$16, R339.1, R342.2
- removed net STEP18: IC38.P$16, R358.1, R361.2
- removed net STEP19: IC40.P$16, R377.1, R380.2
- removed net STEP_IN16: JP202.3, JP204.3, R323.1
- removed net STEP_IN17: JP214.3, JP216.3, R342.1
- removed net STEP_IN18: JP226.3, JP228.3, R361.1
- removed net STEP_IN19: JP238.3, JP240.3, R380.1
- removed net V+16: C145.1, C148.1, C149.1, C151.2, C152.+, D17.C, IC33.IN, IC34.P$22, IC34.P$28
- removed net V+17: C154.1, C157.1, C158.1, C160.2, C161.+, D18.C, IC35.IN, IC36.P$22, IC36.P$28
- removed net V+18: C163.1, C166.1, C167.1, C169.2, C170.+, D19.C, IC37.IN, IC38.P$22, IC38.P$28
- removed net V+19: C172.1, C175.1, C176.1, C178.2, C179.+, D20.C, IC39.IN, IC40.P$22, IC40.P$28
- removed net VCC16: APWR16.2, C147.1, C153.1, IC34.P$15, JP202.1, JP204.1, R307.2, R313.2, R314.2, R315.2, R316.2, R317.2, R319.2, R320.2, R321.1
- removed net VCC17: APWR17.2, C156.1, C162.1, IC36.P$15, JP214.1, JP216.1, R326.2, R332.2, R333.2, R334.2, R335.2, R336.2, R338.2, R339.2, R340.1
- removed net VCC18: APWR18.2, C165.1, C171.1, IC38.P$15, JP226.1, JP228.1, R345.2, R351.2, R352.2, R353.2, R354.2, R355.2, R357.2, R358.2, R359.1
- removed net VCC19: APWR19.2, C174.1, C180.1, IC40.P$15, JP238.1, JP240.1, R364.2, R370.2, R371.2, R372.2, R373.2, R374.2, R376.2, R377.2, R378.1
Routing:
- net V+19: track 58.8 -> 0.00 mm, vias 6 -> 0
- net V+16: track 58.8 -> 0.00 mm, vias 6 -> 0
- net V+18: track 58.8 -> 0.00 mm, vias 6 -> 0
- net V+17: track 58.8 -> 0.00 mm, vias 6 -> 0
- net VCC18: track 34.8 -> 0.00 mm, vias 3 -> 0
- net VCC16: track 34.8 -> 0.00 mm, vias 3 -> 0
- net VCC19: track 34.8 -> 0.00 mm, vias 3 -> 0
- net VCC17: track 34.8 -> 0.00 mm, vias 3 -> 0
- net ENABLE19: track 23.5 -> 0.00 mm, vias 1 -> 0
- net ENABLE16: track 23.5 -> 0.00 mm, vias 1 -> 0
- net ENABLE17: track 23.5 -> 0.00 mm, vias 1 -> 0
- net ENABLE18: track 23.5 -> 0.00 mm, vias 1 -> 0
- net DIR19: track 21.7 -> 0.00 mm, vias 2 -> 0
- net DIR18: track 21.7 -> 0.00 mm, vias 2 -> 0
- net DIR16: track 21.7 -> 0.00 mm, vias 2 -> 0
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- removed copper zone on layer 1, net 5V_ALT16
- removed copper zone on layer 1, net 5V_ALT17
- removed copper zone on layer 1, net 5V_ALT18
- removed copper zone on layer 1, net 5V_ALT19
- removed copper zone on layer 1, net COILA+16
- removed copper zone on layer 16, net COILA+16
- removed copper zone on layer 1, net COILA+17
- removed copper zone on layer 16, net COILA+17
- removed copper zone on layer 1, net COILA+18
- removed copper zone on layer 16, net COILA+18
- removed copper zone on layer 1, net COILA+19
- removed copper zone on layer 16, net COILA+19
- removed copper zone on layer 1, net COILA-16
- removed copper zone on layer 1, net COILA-17
- removed copper zone on layer 1, net COILA-18
- removed copper zone on layer 1, net COILA-19
- removed copper zone on layer 1, net COILB+16
- removed copper zone on layer 16, net COILB+16
- removed copper zone on layer 1, net COILB+17
- removed copper zone on layer 16, net COILB+17
- removed copper zone on layer 1, net COILB+18
- removed copper zone on layer 16, net COILB+18
- removed copper zone on layer 1, net COILB+19
- removed copper zone on layer 16, net COILB+19
- removed copper zone on layer 1, net COILB-16
- removed copper zone on layer 1, net COILB-17
- removed copper zone on layer 1, net COILB-18
- removed copper zone on layer 1, net COILB-19
- removed copper zone on layer 1, net GND16
- removed copper zone on layer 15, net GND16
- removed copper zone on layer 16, net GND16
- removed copper zone on layer 1, net GND17
- removed copper zone on layer 15, net GND17
- removed copper zone on layer 16, net GND17
- removed copper zone on layer 1, net GND18
- removed copper zone on layer 15, net GND18
- removed copper zone on layer 16, net GND18
- removed copper zone on layer 1, net GND19
- removed copper zone on layer 15, net GND19
- removed copper zone on layer 16, net GND19
- removed copper zone on layer 1, net N$244
- removed copper zone on layer 1, net N$245
- removed copper zone on layer 1, net N$259
- removed copper zone on layer 1, net N$260
- removed copper zone on layer 1, net N$274
- removed copper zone on layer 1, net N$275
- removed copper zone on layer 1, net N$289
- removed copper zone on layer 1, net N$290
- removed copper zone on layer 1, net V+16
- removed copper zone on layer 1, net V+17
- removed copper zone on layer 1, net V+18
- removed copper zone on layer 1, net V+19
- removed copper zone on layer 2, net VCC16
- removed copper zone on layer 2, net VCC17
- removed copper zone on layer 2, net VCC18
- removed copper zone on layer 2, net VCC19
Other:
- board size 162.6 x 168.1 mm -> 162.6 x 137.2 mm
- board text added: "v16a"
- board text removed: "This is a 4-layer board!!"
- board text removed: "v16"
