File: Hardware/BigEasyDriver.sch (EAGLE design)
At the start: 55 parts, among them IC1 A4983ALT1, IC2 LM317L

Commit message: Adding 4 layer note to tDocu on board
Other:
- note added: "Produced by SparkFun Electronics"
- note removed: "Produced by Spark Fun Electronics"
Changed lines of the file:
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@@
 <?xml version="1.0" encoding="utf-8"?>
 <!DOCTYPE eagle SYSTEM "eagle.dtd">
-<eagle version="6.5.0">
+<eagle version="6.6.0">
 <drawing>
 <settings>
@@
 <wire x1="111.252" y1="50.8" x2="112.268" y2="50.8" width="0.1524" layer="94"/>
 <text x="169.672" y="11.43" size="1.778" layer="94"> Brian Schmalz</text>
-<text x="148.59" y="6.35" size="1.778" layer="94">Produced by Spark Fun Electronics</text>
+<text x="148.59" y="6.35" size="1.778" layer="94">Produced by SparkFun Electronics</text>
 <text x="142.24" y="53.34" size="1.4224" layer="98">Voltage regulator can supply 100mA</text>
 <text x="71.12" y="58.42" size="1.4224" layer="98">Must use LM317</text>

Commit message: changed fiducials to regulars
also deleted old panels in prep for new ones
Parts:
- removed JP2, JP4: FIDUCIAL1X2.5, abes:FIDUCIAL1X2.5
- added FID1, FID2: FIDUCIAL1X2, SparkFun-Aesthetics:FIDUCIAL1X2
Changed lines of the file:
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@@
 <part name="C2" library="SparkFun-Capacitors" deviceset="1.0UF-16V-10%(0603)" device="" value="1uF"/>
 <part name="LOGO1" library="OSHW" deviceset="OSHW_LOGO_FILL" device="X0100-NT"/>
-<part name="JP2" library="abes" deviceset="FIDUCIAL" device="1X2.5"/>
-<part name="JP4" library="abes" deviceset="FIDUCIAL" device="1X2.5"/>
 <part name="U$3" library="Testing" deviceset="PAD" device=""/>
 <part name="U$4" library="Testing" deviceset="PAD" device=""/>
@@
 <part name="R14" library="SparkFun-Resistors" deviceset="1KOHM1/10W1%(0603)" device="" value="1K"/>
 <part name="R15" library="SparkFun-Resistors" deviceset="1KOHM1/10W1%(0603)" device="" value="1K"/>
+<part name="FID1" library="SparkFun-Aesthetics" deviceset="FIDUCIAL" device="1X2"/>
+<part name="FID2" library="SparkFun-Aesthetics" deviceset="FIDUCIAL" device="1X2"/>
 </parts>
 <sheets>
@@
 <instance part="C2" gate="G$1" x="127" y="35.56"/>
 <instance part="LOGO1" gate="G$1" x="127" y="5.08"/>
-<instance part="JP2" gate="G$1" x="139.7" y="7.62"/>
-<instance part="JP4" gate="G$1" x="134.62" y="7.62"/>
 <instance part="U$3" gate="G$1" x="185.42" y="124.46"/>
 <instance part="U$4" gate="G$1" x="185.42" y="121.92"/>
@@
 <instance part="R14" gate="G$1" x="116.84" y="101.6"/>
 <instance part="R15" gate="G$1" x="116.84" y="93.98"/>
+<instance part="FID1" gate="G$1" x="134.62" y="7.62"/>
+<instance part="FID2" gate="G$1" x="139.7" y="7.62"/>
 </instances>
 <busses>

Commit message: Updating version number to show change in CAM job
Other:
- note added: "BigEasyDriver v1.6a"
- note added: "v16a"
- note removed: "BigEasyDriver v1.6"
- note removed: "v16"
Changed lines of the file:
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@@
 <?xml version="1.0" encoding="utf-8"?>
 <!DOCTYPE eagle SYSTEM "eagle.dtd">
-<eagle version="6.6.0">
+<eagle version="7.1.0">
 <drawing>
 <settings>
@@
 <layer number="254" name="cooling" color="7" fill="1" visible="yes" active="yes"/>
 </layers>
-<schematic>
+<schematic xreflabel="%F%N/%S" xrefpart="/%S.%C%R">
 <attributes>
 </attributes>
@@
 <text x="78.74" y="165.1" size="1.4224" layer="98">Short JP10, or JP6 pins </text>
 <text x="78.74" y="167.64" size="1.4224" layer="98">DEFAULT OPTIONS</text>
-<text x="2.54" y="177.8" size="5.08" layer="98">BigEasyDriver v1.6</text>
+<text x="2.54" y="177.8" size="5.08" layer="98">BigEasyDriver v1.6a</text>
 <text x="5.08" y="99.06" size="1.4224" layer="98">DIR is level sensitive</text>
 <text x="5.08" y="96.52" size="1.4224" layer="98">A rising edge on STEP</text>
@@
 <text x="5.08" y="16.51" size="0.8128" layer="98">-ran all traces directly away from IC</text>
 <text x="5.08" y="15.24" size="0.8128" layer="98">-moved vias and retraced as necessary on VCC and TOP layers</text>
-<text x="238.76" y="7.62" size="2.54" layer="94" font="vector">v16</text>
+<text x="238.76" y="7.62" size="2.54" layer="94" font="vector">v16a</text>
 <text x="148.59" y="8.89" size="1.778" layer="94">Revised by Patrick Alberts</text>
 <text x="2.54" y="13.97" size="0.8128" layer="98">v1.4 SF 4/17/2013 Fixed current adjustment pot silk so directions are correct</text>

Commit message: Updating IC to proper A4988 device
Parts:
- IC1: value A4983ALT1 -> A4988ALT1; device Testing:A4983ALT1 -> SparkFun-PowerIC:A4988ALT1
Changed lines of the file:
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@@
 <?xml version="1.0" encoding="utf-8"?>
 <!DOCTYPE eagle SYSTEM "eagle.dtd">
-<eagle version="7.1.0">
+<eagle version="7.2.0">
 <drawing>
 <settings>
@@
 <layer number="54" name="bGND_GNDA" color="1" fill="9" visible="no" active="no"/>
 <layer number="56" name="wert" color="7" fill="1" visible="no" active="no"/>
+<layer number="57" name="tCAD" color="7" fill="1" visible="no" active="no"/>
+<layer number="59" name="tCarbon" color="7" fill="1" visible="no" active="no"/>
+<layer number="60" name="bCarbon" color="7" fill="1" visible="no" active="no"/>
+<layer number="90" name="Modules" color="5" fill="1" visible="yes" active="yes"/>
 <layer number="91" name="Nets" color="2" fill="1" visible="yes" active="yes"/>
 <layer number="92" name="Busses" color="1" fill="1" visible="yes" active="yes"/>
@@
 <layer number="97" name="Info" color="7" fill="1" visible="yes" active="yes"/>
 <layer number="98" name="Guide" color="6" fill="1" visible="yes" active="yes"/>
+<layer number="99" name="SpiceOrder" color="7" fill="1" visible="yes" active="yes"/>
 <layer number="100" name="Muster" color="7" fill="1" visible="no" active="no"/>
 <layer number="101" name="Patch_Top" color="12" fill="4" visible="yes" active="yes"/>
@@
 <layer number="108" name="tplace-old" color="10" fill="1" visible="yes" active="yes"/>
 <layer number="109" name="ref-old" color="11" fill="1" visible="yes" active="yes"/>
+<layer number="110" name="fp0" color="7" fill="1" visible="yes" active="yes"/>
+<layer number="111" name="LPC17xx" color="7" fill="1" visible="yes" active="yes"/>
+<layer number="112" name="tSilk" color="7" fill="1" visible="yes" active="yes"/>
+<layer number="113" name="IDFDebug" color="4" fill="1" visible="yes" active="yes"/>
 <layer number="116" name="Patch_BOT" color="9" fill="4" visible="yes" active="yes"/>
+<layer number="118" name="Rect_Pads" color="7" fill="1" visible="yes" active="yes"/>
 <layer number="121" name="_tsilk" color="7" fill="1" visible="yes" active="yes"/>
 <layer number="122" name="_bsilk" color="7" fill="1" visible="yes" active="yes"/>
+<layer number="123" name="tTestmark" color="7" fill="1" visible="yes" active="yes"/>
+<layer number="124" name="bTestmark" color="7" fill="1" visible="yes" active="yes"/>
 <layer number="125" name="_tNames" color="7" fill="1" visible="yes" active="yes"/>
+<layer number="126" name="_bNames" color="7" fill="1" visible="yes" active="yes"/>
+<layer number="127" name="_tValues" color="7" fill="1" visible="yes" active="yes"/>
+<layer number="128" name="_bValues" color="7" fill="1" visible="yes" active="yes"/>
+<layer number="129" name="Mask" color="7" fill="1" visible="yes" active="yes"/>
+<layer number="131" name="tAdjust" color="7" fill="1" visible="yes" active="yes"/>
+<layer number="132" name="bAdjust" color="7" fill="1" visible="yes" active="yes"/>
 <layer number="144" name="DrillLegend" color="7" fill="1" visible="yes" active="yes"/>
+<layer number="150" name="Notes" color="7" fill="1" visible="yes" active="yes"/>
 <layer number="151" name="HeatSink" color="7" fill="1" visible="yes" active="yes"/>
+<layer number="152" name="_bDocu" color="7" fill="1" visible="yes" active="yes"/>
+<layer number="153" name="FabDoc1" color="7" fill="1" visible="yes" active="yes"/>
+<layer number="154" name="FabDoc2" color="7" fill="1" visible="yes" active="yes"/>
+<layer number="155" name="FabDoc3" color="7" fill="1" visible="yes" active="yes"/>
 <layer number="199" name="Contour" color="7" fill="1" visible="yes" active="yes"/>
 <layer number="200" name="200bmp" color="1" fill="10" visible="no" active="no"/>
@@
 <layer number="223" name="223bmp" color="24" fill="1" visible="no" active="no"/>
 <layer number="224" name="224bmp" color="25" fill="1" visible="no" active="no"/>
+<layer number="225" name="225bmp" color="7" fill="1" visible="yes" active="yes"/>
+<layer number="226" name="226bmp" color="7" fill="1" visible="yes" active="yes"/>
+<layer number="227" name="227bmp" color="7" fill="1" visible="yes" active="yes"/>
+<layer number="228" name="228bmp" color="7" fill="1" visible="yes" active="yes"/>
+<layer number="229" name="229bmp" color="7" fill="1" visible="yes" active="yes"/>
+<layer number="230" name="230bmp" color="7" fill="1" visible="yes" active="yes"/>
+<layer number="231" name="231bmp" color="7" fill="1" visible="yes" active="yes"/>
+<layer number="248" name="Housing" color="7" fill="1" visible="yes" active="yes"/>
+<layer number="249" name="Edge" color="7" fill="1" visible="yes" active="yes"/>
 <layer number="250" name="Descript" color="3" fill="1" visible="no" active="no"/>
 <layer number="251" name="SMDround" color="12" fill="11" visible="no" active="no"/>
 <layer number="254" name="cooling" color="7" fill="1" visible="yes" active="yes"/>
+<layer number="255" name="routoute" color="7" fill="1" visible="yes" active="yes"/>
 </layers>
-<schematic xreflabel="%F%N/%S" xrefpart="/%S.%C%R">
+<schematic xreflabel="%F%N/%S" xrefpart="/%S">
 <attributes>
 </attributes>
@@
 <part name="R18" library="SparkFun-Resistors" deviceset="0.11OHM1/2W1%(2010)" device="" value=".11"/>
 <part name="R19" library="SparkFun-Resistors" deviceset="0.11OHM1/2W1%(2010)" device="" value=".11"/>
-<part name="IC1" library="Testing" deviceset="A4983" device="ALT1"/>
+<part name="IC1" library="SparkFun-PowerIC" deviceset="A4988" device="ALT1"/>
 <part name="GND16" library="supply1" deviceset="GND" device=""/>
 <part name="R20" library="SparkFun-Resistors" deviceset="20KOHM1/10W5%(0603)" device="" value="20K"/>

Commit message: Fixing typo in schematic note to proper screw terminal size
Other:
- note added: "3.5mm Screw Terminals"
- note removed: "2.5mm Screw Terminals"
Changed lines of the file:
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@@
 <?xml version="1.0" encoding="utf-8"?>
 <!DOCTYPE eagle SYSTEM "eagle.dtd">
-<eagle version="7.2.0">
+<eagle version="7.7.0">
 <drawing>
 <settings>
@@
 <text x="71.628" y="137.16" size="1.4224" layer="98">D.N.I</text>
 <text x="41.656" y="139.954" size="1.4224" layer="98">.100" Headers</text>
-<text x="71.628" y="139.7" size="1.4224" layer="98">2.5mm Screw Terminals</text>
+<text x="71.628" y="139.7" size="1.4224" layer="98">3.5mm Screw Terminals</text>
 <text x="2.54" y="22.86" size="0.8128" layer="98">v1.1 BPS Added pull-ups, re-routed</text>
 <text x="2.54" y="81.28" size="1.4224" layer="98">Bi-polar Stepper Motor Outputs</text>
